File: KICAD/Energy_Meter_V3/Energy_Meter_V3.kicad_sch (KiCad schematic)
At the start: 134 parts, among them J1 Conn_01x02_Pin, J10 Barrel_Jack_Switch_Pin3Ring, J2 Conn_01x02_Pin, J3 Conn_01x02_Pin, J4 Conn_01x04_Socket, J6 Conn_01x04_Socket, J7 USB_C_Receptacle_USB2.0_16P, J8 USB_C_Receptacle_USB2.0_16P, J9 Conn_01x04_Socket, U1 ADE7758, U10 STM32F103C8Tx, U2 AMS1117-5.0, U3 PC817, U4 TME-0505S, U5 XL1509-5.0, U6 ESP32-C3-WROOM-02U, Y2 32.768k, Y3 8M, Y4 10M, Y5 32.768k

Commit message: update 50%
Parts:
- removed C21: 4.7uF, Capacitor_SMD:CP_Elec_4x5.4, symbol Device:C_Polarized
- removed C22, C23: 100nF, Capacitor_SMD:C_0603_1608Metric_Pad1.08x0.95mm_HandSolder, symbol Device:C
- removed C24: 10uF, Capacitor_SMD:CP_Elec_4x5.4, symbol Device:C_Polarized
- removed L2, L4: 4.7uH, Inductor_SMD:L_1206_3216Metric_Pad1.22x1.90mm_HandSolder, symbol Device:L
- removed U4: TME-0505S, Converter_DCDC:Converter_DCDC_TRACO_TME_03xxS_05xxS_12xxS_Single_THT, symbol Converter_DCDC:TME-1205S
- R1: renamed from R7; footprint Resistor_SMD:R_0805_2012Metric_Pad1.20x1.40mm_HandSolder -> Resistor_SMD:R_0603_1608Metric_Pad0.98x0.95mm_HandSolder
- R10: renamed from R14; footprint Resistor_SMD:R_0805_2012Metric_Pad1.20x1.40mm_HandSolder -> Resistor_SMD:R_0603_1608Metric_Pad0.98x0.95mm_HandSolder
- R11: renamed from R20; footprint Resistor_SMD:R_0805_2012Metric_Pad1.20x1.40mm_HandSolder -> Resistor_SMD:R_0603_1608Metric_Pad0.98x0.95mm_HandSolder
- R12: renamed from R23; footprint Resistor_SMD:R_0805_2012Metric_Pad1.20x1.40mm_HandSolder -> Resistor_SMD:R_0603_1608Metric_Pad0.98x0.95mm_HandSolder
- R13: renamed from R26; footprint Resistor_SMD:R_0805_2012Metric_Pad1.20x1.40mm_HandSolder -> Resistor_SMD:R_0603_1608Metric_Pad0.98x0.95mm_HandSolder
- R14: renamed from R5; footprint Resistor_SMD:R_0805_2012Metric_Pad1.20x1.40mm_HandSolder -> Resistor_SMD:R_0603_1608Metric_Pad0.98x0.95mm_HandSolder
- R15, R8, R9: footprint Resistor_SMD:R_0805_2012Metric_Pad1.20x1.40mm_HandSolder -> Resistor_SMD:R_0603_1608Metric_Pad0.98x0.95mm_HandSolder
- R16: renamed from R2; footprint Resistor_SMD:R_0805_2012Metric_Pad1.20x1.40mm_HandSolder -> Resistor_SMD:R_0603_1608Metric_Pad0.98x0.95mm_HandSolder
- R17: renamed from R10; footprint Resistor_SMD:R_0805_2012Metric_Pad1.20x1.40mm_HandSolder -> Resistor_SMD:R_0603_1608Metric_Pad0.98x0.95mm_HandSolder
- R18: renamed from R16; footprint Resistor_SMD:R_0805_2012Metric_Pad1.20x1.40mm_HandSolder -> Resistor_SMD:R_0603_1608Metric_Pad0.98x0.95mm_HandSolder
- R19: renamed from R11; footprint Resistor_SMD:R_0805_2012Metric_Pad1.20x1.40mm_HandSolder -> Resistor_SMD:R_0603_1608Metric_Pad0.98x0.95mm_HandSolder
- R2: renamed from R30; footprint Resistor_SMD:R_0805_2012Metric_Pad1.20x1.40mm_HandSolder -> Resistor_SMD:R_0603_1608Metric_Pad0.98x0.95mm_HandSolder
- R20: renamed from R6; footprint Resistor_SMD:R_0805_2012Metric_Pad1.20x1.40mm_HandSolder -> Resistor_SMD:R_0603_1608Metric_Pad0.98x0.95mm_HandSolder
- R21: renamed from R17; footprint Resistor_SMD:R_0805_2012Metric_Pad1.20x1.40mm_HandSolder -> Resistor_SMD:R_0603_1608Metric_Pad0.98x0.95mm_HandSolder
- R22: renamed from R3; footprint Resistor_SMD:R_0805_2012Metric_Pad1.20x1.40mm_HandSolder -> Resistor_SMD:R_0603_1608Metric_Pad0.98x0.95mm_HandSolder
- R23: renamed from R22; footprint Resistor_SMD:R_0805_2012Metric_Pad1.20x1.40mm_HandSolder -> Resistor_SMD:R_0603_1608Metric_Pad0.98x0.95mm_HandSolder
- R24: renamed from R25; footprint Resistor_SMD:R_0805_2012Metric_Pad1.20x1.40mm_HandSolder -> Resistor_SMD:R_0603_1608Metric_Pad0.98x0.95mm_HandSolder
- R25: renamed from R28; footprint Resistor_SMD:R_0805_2012Metric_Pad1.20x1.40mm_HandSolder -> Resistor_SMD:R_0603_1608Metric_Pad0.98x0.95mm_HandSolder
- R26: renamed from R12; footprint Resistor_SMD:R_0805_2012Metric_Pad1.20x1.40mm_HandSolder -> Resistor_SMD:R_0603_1608Metric_Pad0.98x0.95mm_HandSolder
- R27: renamed from R19; footprint Resistor_SMD:R_0805_2012Metric_Pad1.20x1.40mm_HandSolder -> Resistor_SMD:R_0603_1608Metric_Pad0.98x0.95mm_HandSolder
- R28: renamed from R18; footprint Resistor_SMD:R_0805_2012Metric_Pad1.20x1.40mm_HandSolder -> Resistor_SMD:R_0603_1608Metric_Pad0.98x0.95mm_HandSolder
- R3: renamed from R4; footprint Resistor_SMD:R_0805_2012Metric_Pad1.20x1.40mm_HandSolder -> Resistor_SMD:R_0603_1608Metric_Pad0.98x0.95mm_HandSolder
- R4: renamed from R31; footprint Resistor_SMD:R_0805_2012Metric_Pad1.20x1.40mm_HandSolder -> Resistor_SMD:R_0603_1608Metric_Pad0.98x0.95mm_HandSolder
- R43: renamed from R21; footprint Resistor_SMD:R_0805_2012Metric_Pad1.20x1.40mm_HandSolder -> Resistor_SMD:R_0603_1608Metric_Pad0.98x0.95mm_HandSolder
- R47: renamed from R24; footprint Resistor_SMD:R_0805_2012Metric_Pad1.20x1.40mm_HandSolder -> Resistor_SMD:R_0603_1608Metric_Pad0.98x0.95mm_HandSolder
- R5: renamed from R13; footprint Resistor_SMD:R_0805_2012Metric_Pad1.20x1.40mm_HandSolder -> Resistor_SMD:R_0603_1608Metric_Pad0.98x0.95mm_HandSolder
- R6: renamed from R32; footprint Resistor_SMD:R_0805_2012Metric_Pad1.20x1.40mm_HandSolder -> Resistor_SMD:R_0603_1608Metric_Pad0.98x0.95mm_HandSolder
- R7: renamed from R1; footprint Resistor_SMD:R_0805_2012Metric_Pad1.20x1.40mm_HandSolder -> Resistor_SMD:R_0603_1608Metric_Pad0.98x0.95mm_HandSolder
- renumbered RST2 to BUT1, C3 to C1, C6 to C10, C65 to C11, C14 to C12, C69 to C14, C57 to C15, C62 to C16, C58 to C17, C59 to C18, C15 to C19, C63 to C20, C60 to C21, C16 to C22, C11 to C23, C12 to C24, C61 to C25, C64 to C26, C66 to C27, C67 to C28, C25 to C29, C5 to C3, C26 to C30, C74 to C31, C73 to C32, C27 to C33, C68 to C34, C19 to C35, C70 to C36, C20 to C37, C71 to C38, C75 to C39, C7 to C4, C17 to C40, C72 to C41, C76 to C42, C18 to C43, C8 to C5, C9 to C6, C10 to C7, C1 to C8, C4 to C9, D2 to D1, D4 to D2, D1 to D4, RST3 to EN1, J4 to J1, J1 to J2, J2 to J3, J3 to J4, J9 to J5, J10 to J7, J7 to J9, JP5 to JP1, JP7 to JP2, JP1 to JP3, JP2 to JP4, L3 to L1, R33 to R29, R37 to R30, R39 to R31, R34 to R32, R38 to R33, R36 to R34, R44 to R36, R42 to R37, R43 to R38, R41 to R39, R58 to R40, R40 to R41, R27 to R42, R59 to R44, R60 to R45, R29 to R46, TP6 to TP1, TP7 to TP2, TP8 to TP3, U3 to U2, U10 to U3, U5 to U4, U2 to U5, Y4 to Y1, Y5 to Y4
Connections:
- net IO1 is gone; now on net IO3: LED_ESP1.1 (K)
- net RESET: no longer BUT1.1, C32.2, R41.2
- net IO3: now reaches U6.15 (IO3)
- net IO4: now reaches U6.3 (IO4)
- net IO4: now also BUT1.1, C32.2, R41.2
Other:
- moved on the sheet: BUT1, C14, C27, C28, C29, C30, C31, C32, C33, C34, C35, C36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

Commit message: update 70%
Parts:
- removed JP1, JP2: Jumper_2_Open, Connector_PinHeader_2.54mm:PinHeader_1x02_P2.54mm_Vertical, symbol Jumper:Jumper_2_Open
- removed U2: PC817, Package_DIP:DIP-4_W7.62mm, symbol Isolator:PC817
- added Q1: Q_NPN_BEC, Package_TO_SOT_SMD:SOT-23, symbol Transistor_BJT:Q_NPN_BEC
Connections:
- net +5V: now also C12.1, C13.1, U1.3 (DVDD), U1.4 (AVDD)
- net DIN: no longer U3.31 (PA10)
- net GND1: now also Q1.2 (E)
- net PA3: now also Q1.3 (C)
- net UART1_RX: now also U3.30 (PA9); no longer U3.29 (PA8)
- net UART1_TX: now also U3.31 (PA10); no longer U3.30 (PA9)
- net at R32.1: now also Q1.1 (B)

Commit message: upload 80%
Parts:
- J8, J9: footprint Connector_USB:USB_C_Receptacle_GCT_USB4110 -> Connector_USB:USB_C_Receptacle_Palconn_UTC16-G
Connections:
- net A: now also J1.1 (Pin_1); no longer J1.4 (Pin_4)
- net B: now also J1.2 (Pin_2); no longer J1.3 (Pin_3)
- net C: now also J1.3 (Pin_3); no longer J1.2 (Pin_2)
- net N: now also J1.4 (Pin_4); no longer J1.1 (Pin_1)
Other:
- moved on the sheet: J1
Changed lines of the file:
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@@
 	(wire
 		(pts
-			(xy 21.59 127) (xy 27.94 127)
-		)
-		(stroke
-			(width 0)
-			(type default)
-		)
-	)
-	(wire
-		(pts
 			(xy 55.88 161.29) (xy 55.88 162.56)
 		)
@@
 	(wire
 		(pts
-			(xy 60.96 121.92) (xy 64.77 121.92)
+			(xy 21.59 121.92) (xy 53.34 121.92)
 		)
 		(stroke
@@
 	(wire
 		(pts
-			(xy 109.22 124.46) (xy 109.22 127)
+			(xy 60.96 121.92) (xy 64.77 121.92)
 		)
 		(stroke
@@
 	(wire
 		(pts
-			(xy 105.41 60.96) (xy 109.22 60.96)
+			(xy 109.22 124.46) (xy 109.22 127)
 		)
 		(stroke
@@
 	(wire
 		(pts
-			(xy 203.2 39.37) (xy 203.2 41.91)
+			(xy 105.41 60.96) (xy 109.22 60.96)
 		)
 		(stroke
@@
 	(wire
 		(pts
-			(xy 355.6 229.87) (xy 361.95 229.87)
+			(xy 203.2 39.37) (xy 203.2 41.91)
 		)
 		(stroke
@@
 	(wire
 		(pts
-			(xy 41.91 161.29) (xy 55.88 161.29)
+			(xy 355.6 229.87) (xy 361.95 229.87)
 		)
 		(stroke
@@
 	(wire
 		(pts
-			(xy 322.58 83.82) (xy 331.47 83.82)
+			(xy 41.91 161.29) (xy 55.88 161.29)
 		)
 		(stroke
@@
 	(wire
 		(pts
-			(xy 115.57 171.45) (xy 115.57 173.99)
+			(xy 322.58 83.82) (xy 331.47 83.82)
 		)
 		(stroke
@@
 	(wire
 		(pts
-			(xy 21.59 121.92) (xy 53.34 121.92)
+			(xy 115.57 171.45) (xy 115.57 173.99)
 		)
 		(stroke
@@
 	(wire
 		(pts
-			(xy 25.4 124.46) (xy 21.59 124.46)
-		)
-		(stroke
-			(width 0)
-			(type default)
-		)
-	)
-	(wire
-		(pts
 			(xy 27.94 62.23) (xy 27.94 63.5)
 		)
@@
 	(wire
 		(pts
+			(xy 21.59 127) (xy 27.94 127)
+		)
+		(stroke
+			(width 0)
+			(type default)
+		)
+	)
+	(wire
+		(pts
 			(xy 21.59 129.54) (xy 30.48 129.54)
 		)
@@
 	(wire
 		(pts
+			(xy 21.59 124.46) (xy 25.4 124.46)
+		)
+		(stroke
+			(width 0)
+			(type default)
+		)
+	)
+	(wire
+		(pts
 			(xy 68.58 69.85) (xy 68.58 72.39)
 		)
@@
 			)
 		)
-		(property "Footprint" "Connector_USB:USB_C_Receptacle_GCT_USB4110"
+		(property "Footprint" "Connector_USB:USB_C_Receptacle_Palconn_UTC16-G"
 			(at 377.19 140.97 0)
 			(hide yes)
@@
 			)
 		)
-		(property "Footprint" "Connector_USB:USB_C_Receptacle_GCT_USB4110"
+		(property "Footprint" "Connector_USB:USB_C_Receptacle_Palconn_UTC16-G"
 			(at 250.19 140.97 0)
 			(hide yes)
@@
 	(symbol
 		(lib_id "Connector:Conn_01x04_Socket")
-		(at 16.51 124.46 0)
-		(mirror y)
+		(at 16.51 127 180)
 		(unit 1)
 		(body_style 1)
@@
 		(dnp no)
 		(property "Reference" "J1"
-			(at 20.574 132.588 0)
+			(at 20.574 118.872 0)
 			(show_name no)
 			(do_not_autoplace no)
@@
 		)
 		(property "Value" "Conn_01x04_Socket"
-			(at 34.798 136.144 0)
+			(at 34.798 115.316 0)
 			(show_name no)
 			(do_not_autoplace no)
@@
 		)
 		(property "Footprint" "TerminalBlock_Phoenix:TerminalBlock_Phoenix_MKDS-1,5-4_1x04_P5.00mm_Horizontal"
-			(at 16.51 124.46 0)
+			(at 16.51 127 0)
 			(hide yes)
 			(show_name no)
@@
 		)
 		(property "Datasheet" ""
-			(at 16.51 124.46 0)
+			(at 16.51 127 0)
 			(hide yes)
 			(show_name no)
@@
 		)
 		(property "Description" "Generic connector, single row, 01x04, script generated"
-			(at 16.51 124.46 0)
+			(at 16.51 127 0)
 			(hide yes)
 			(show_name no)
