File: KICAD/Energy_Meter_V3/Energy_Meter_V3.kicad_pcb (KiCad board)
At the start: 2 copper layers, 92 x 86 mm, 99 parts, among them J1 Conn_01x02_Pin, J2 Conn_01x02_Pin, J3 Conn_01x02_Pin, J4 Conn_01x04_Socket, J5 Jack-DC, J6 Conn_01x04_Socket, J9 USB_C_Receptacle_PowerOnly_6P, U1 ADE7758, U10 STM32F103C8Tx, U2 AMS1117-5.0, U3 PC817, U4 TME-1205S, U5 ESP32-C3_SUPERMINI_TH, Y2 32.768k, Y3 8M, Y4 10M

Commit message: update 50%
Parts:
- removed C57, C58, C59, C60, C69: 100n, Capacitor_SMD:C_0603_1608Metric_Pad1.08x0.95mm_HandSolder
- removed C61, C64: 10p, Capacitor_SMD:C_0603_1608Metric_Pad1.08x0.95mm_HandSolder
- removed C62, C63, C65: 100p, Capacitor_SMD:C_0603_1608Metric_Pad1.08x0.95mm_HandSolder
- removed C66, C67: 12p, Capacitor_SMD:C_0603_1608Metric_Pad1.08x0.95mm_HandSolder
- removed JP5, JP7: Jumper_2_Open, Connector_PinHeader_2.54mm:PinHeader_1x02_P2.54mm_Vertical
- removed L2, L4: 4.7uH, Inductor_SMD:L_1206_3216Metric_Pad1.22x1.90mm_HandSolder
- removed R58: 4.7k, Resistor_SMD:R_0603_1608Metric_Pad0.98x0.95mm_HandSolder
- removed U10: STM32F103C8Tx, Package_QFP:LQFP-48_7x7mm_P0.5mm
- added BUT1: SW_Push, Button_Switch_SMD:SW_SPST_CK_RS282G05A3, F.Cu at (155.4, 74.0)
- added C17: 100n, Capacitor_SMD:C_0603_1608Metric_Pad1.08x0.95mm_HandSolder, F.Cu at (97.2, 55.7)
- added C18: 100n, Capacitor_SMD:C_0603_1608Metric_Pad1.08x0.95mm_HandSolder, F.Cu at (97.2, 57.2)
- added C25: 10p, Capacitor_SMD:C_0603_1608Metric_Pad1.08x0.95mm_HandSolder, F.Cu at (83.4, 64.6)
- added C26: 10p, Capacitor_SMD:C_0603_1608Metric_Pad1.08x0.95mm_HandSolder, F.Cu at (83.4, 70.4)
- added C27: 12p, Capacitor_SMD:C_0603_1608Metric_Pad1.08x0.95mm_HandSolder, F.Cu at (83.4, 60.6)
- added C28: 12p, Capacitor_SMD:C_0603_1608Metric_Pad1.08x0.95mm_HandSolder, F.Cu at (83.4, 63.1)
- added C29: 100n, Capacitor_SMD:C_0603_1608Metric_Pad1.08x0.95mm_HandSolder, F.Cu at (153.4, 44.5)
- added C30: 220u, Capacitor_SMD:CP_Elec_6.3x7.7, F.Cu at (150.6, 48.8)
- added C31: 100p, Capacitor_SMD:C_0603_1608Metric_Pad1.08x0.95mm_HandSolder, F.Cu at (158.5, 69.8)
- added C32: 100p, Capacitor_SMD:C_0603_1608Metric_Pad1.08x0.95mm_HandSolder, F.Cu at (158.5, 77.0)
- added C33: 100n, Capacitor_SMD:C_0603_1608Metric_Pad1.08x0.95mm_HandSolder, F.Cu at (131.1, 54.6)
- added C34: 10u, Capacitor_SMD:C_0603_1608Metric_Pad1.08x0.95mm_HandSolder, F.Cu at (158.5, 93.7)
- added C35: 10u, Capacitor_SMD:CP_Elec_4x5.4, F.Cu at (121.3, 65.8)
- added C36: 1u, Capacitor_SMD:C_0603_1608Metric_Pad1.08x0.95mm_HandSolder, F.Cu at (158.5, 95.2)
- added C37: 100n, Capacitor_SMD:C_0603_1608Metric_Pad1.08x0.95mm_HandSolder, F.Cu at (117.2, 63.4)
- added C38: 100n, Capacitor_SMD:C_0603_1608Metric_Pad1.08x0.95mm_HandSolder, F.Cu at (158.5, 96.7)
- added C39: 12p, Capacitor_SMD:C_0603_1608Metric_Pad1.08x0.95mm_HandSolder, F.Cu at (132.5, 91.0)
- added C40: 33n, Capacitor_SMD:C_0603_1608Metric_Pad1.08x0.95mm_HandSolder, F.Cu at (142.5, 75.1)
- added C41: 100n, Capacitor_SMD:C_0603_1608Metric_Pad1.08x0.95mm_HandSolder, F.Cu at (158.5, 98.2)
- added C42: 12p, Capacitor_SMD:C_0603_1608Metric_Pad1.08x0.95mm_HandSolder, F.Cu at (132.5, 88.5)
- added C43: 33n, Capacitor_SMD:C_0603_1608Metric_Pad1.08x0.95mm_HandSolder, F.Cu at (147.0, 75.1)
- added D4: LED, LED_SMD:LED_0805_2012Metric_Pad1.15x1.40mm_HandSolder, F.Cu at (144.8, 175.4)
- added EN1: SW_Push, Button_Switch_SMD:SW_SPST_CK_RS282G05A3, F.Cu at (155.5, 66.9)
- added J7: Barrel_Jack_Switch_Pin3Ring, Connector_BarrelJack:BarrelJack_Kycon_KLDX-0202-xC_Horizontal, F.Cu at (141.9, 51.5)
- added J8: USB_C_Receptacle_USB2.0_16P, Connector_USB:USB_C_Receptacle_GCT_USB4110, F.Cu at (107.8, 41.2)
- added JP3: Jumper_3_Bridged12, Connector_PinHeader_2.54mm:PinHeader_1x03_P2.54mm_Vertical, F.Cu at (88.1, 51.5)
- added JP4: Jumper_3_Bridged12, Connector_PinHeader_2.54mm:PinHeader_1x03_P2.54mm_Vertical, F.Cu at (88.1, 47.9)
- added L1: 68uH/2A, Inductor_SMD:L_Bourns_SRP7028A_7.3x6.6mm, F.Cu at (132.9, 61.4)
- added LED1: LED, LED_SMD:LED_0805_2012Metric_Pad1.15x1.40mm_HandSolder, F.Cu at (139.3, 64.8)
- added R21: 1k, Resistor_SMD:R_0603_1608Metric_Pad0.98x0.95mm_HandSolder, F.Cu at (115.3, 100.5)
- added R24: 1k, Resistor_SMD:R_0603_1608Metric_Pad0.98x0.95mm_HandSolder, F.Cu at (136.0, 103.9)
- added R27: 1k, Resistor_SMD:R_0603_1608Metric_Pad0.98x0.95mm_HandSolder, F.Cu at (144.5, 103.9)
- added R40: 4.7k, Resistor_SMD:R_0603_1608Metric_Pad0.98x0.95mm_HandSolder, F.Cu at (134.3, 86.5)
- added R41: 10k, Resistor_SMD:R_0603_1608Metric_Pad0.98x0.95mm_HandSolder, F.Cu at (155.1, 77.0)
- added R42: 5.1k, Resistor_SMD:R_0603_1608Metric_Pad0.98x0.95mm_HandSolder, F.Cu at (131.1, 65.8)
- added R43: 0, Resistor_SMD:R_0603_1608Metric_Pad0.98x0.95mm_HandSolder, F.Cu at (144.0, 75.1)
- added R44: 0, Resistor_SMD:R_0603_1608Metric_Pad0.98x0.95mm_HandSolder, F.Cu at (138.2, 91.0)
- added R45: 0, Resistor_SMD:R_0603_1608Metric_Pad0.98x0.95mm_HandSolder, F.Cu at (138.2, 89.5)
- added R46: 2k, Resistor_SMD:R_0603_1608Metric_Pad0.98x0.95mm_HandSolder, F.Cu at (114.9, 156.5)
- added R47: 0, Resistor_SMD:R_0603_1608Metric_Pad0.98x0.95mm_HandSolder, F.Cu at (145.5, 75.1)
- added TP1: 12V_PWR, TestPoint:TestPoint_Loop_D1.80mm_Drill1.0mm_Beaded, F.Cu at (238.9, 52.9)
- added TP2: GND_PWR, TestPoint:TestPoint_Loop_D1.80mm_Drill1.0mm_Beaded, F.Cu at (238.9, 57.5)
- added TP3: 5V_PWR, TestPoint:TestPoint_Loop_D1.80mm_Drill1.0mm_Beaded, F.Cu at (238.9, 62.1)
- added U6: ESP32-C3-WROOM-02U, RF_Module:ESP32-C3-WROOM-02U, F.Cu at (150.6, 85.0)
- added Y1: 10M, Crystal:Crystal_SMD_5032-4Pin_5.0x3.2mm, F.Cu at (101.9, 77.8)
- C11: value 22p -> 100p
- C12: value 22p -> 10u; footprint Capacitor_SMD:C_0603_1608Metric_Pad1.08x0.95mm_HandSolder -> Capacitor_Tantalum_SMD:CP_EIA-3216-10_Kemet-I_HandSolder
- C14, C15: value 10u -> 100n; footprint Capacitor_Tantalum_SMD:CP_EIA-3216-10_Kemet-I_HandSolder -> Capacitor_SMD:C_0603_1608Metric_Pad1.08x0.95mm_HandSolder
- C16, C20: value 100n -> 100p
- C19: footprint Capacitor_SMD:CP_Elec_4x5.4 -> Capacitor_Tantalum_SMD:CP_EIA-3216-10_Kemet-I_HandSolder
- C21: value 4.7uF -> 100n; footprint Capacitor_SMD:CP_Elec_4x5.4 -> Capacitor_SMD:C_0603_1608Metric_Pad1.08x0.95mm_HandSolder
- C22: value 100nF -> 100n
- C23: value 100nF -> 22p
- C24: value 10uF -> 22p; footprint Capacitor_SMD:CP_Elec_4x5.4 -> Capacitor_SMD:C_0603_1608Metric_Pad1.08x0.95mm_HandSolder
- D2: value LED -> D_Schottky; footprint LED_SMD:LED_0805_2012Metric_Pad1.15x1.40mm_HandSolder -> Diode_SMD:D_SMA_Handsoldering
- J1: value Conn_01x02_Pin -> Conn_01x04_Socket; footprint TerminalBlock_Phoenix:TerminalBlock_Phoenix_MKDS-1,5-2_1x02_P5.00mm_Horizontal -> TerminalBlock_Phoenix:TerminalBlock_Phoenix_MKDS-1,5-4_1x04_P5.00mm_Horizontal
- J4: value Conn_01x04_Socket -> Conn_01x02_Pin; footprint TerminalBlock_Phoenix:TerminalBlock_Phoenix_MKDS-1,5-4_1x04_P5.00mm_Horizontal -> TerminalBlock_Phoenix:TerminalBlock_Phoenix_MKDS-1,5-2_1x02_P5.00mm_Horizontal
- J5: value Jack-DC -> Conn_01x04_Socket; footprint Connector_BarrelJack:BarrelJack_GCT_DCJ200-10-A_Horizontal -> Connector_PinHeader_2.54mm:PinHeader_1x04_P2.54mm_Vertical
- J9: value USB_C_Receptacle_PowerOnly_6P -> USB_C_Receptacle_USB2.0_16P; footprint Connector_USB:USB_C_Receptacle_GCT_USB4125-xx-x_6P_TopMnt_Horizontal -> Connector_USB:USB_C_Receptacle_GCT_USB4110
- JP1, JP2: value Jumper_3_Bridged12 -> Jumper_2_Open; footprint Connector_PinHeader_2.54mm:PinHeader_1x03_P2.54mm_Vertical -> Connector_PinHeader_2.54mm:PinHeader_1x02_P2.54mm_Vertical
- R1, R15, R16, R19, R22, R25, R28, R7, R8, R9: footprint Resistor_SMD:R_0805_2012Metric_Pad1.20x1.40mm_HandSolder -> Resistor_SMD:R_0603_1608Metric_Pad0.98x0.95mm_HandSolder
- R10, R5: value 100 -> 8; footprint Resistor_SMD:R_0805_2012Metric_Pad1.20x1.40mm_HandSolder -> Resistor_SMD:R_0603_1608Metric_Pad0.98x0.95mm_HandSolder
- R11, R12: value 1k -> 500k; footprint Resistor_SMD:R_0805_2012Metric_Pad1.20x1.40mm_HandSolder -> Resistor_SMD:R_0603_1608Metric_Pad0.98x0.95mm_HandSolder
- R13: value 8 -> 500k; footprint Resistor_SMD:R_0805_2012Metric_Pad1.20x1.40mm_HandSolder -> Resistor_SMD:R_0603_1608Metric_Pad0.98x0.95mm_HandSolder
- R14: value 8 -> 100; footprint Resistor_SMD:R_0805_2012Metric_Pad1.20x1.40mm_HandSolder -> Resistor_SMD:R_0603_1608Metric_Pad0.98x0.95mm_HandSolder
- R17, R18: value 1k -> 100; footprint Resistor_SMD:R_0805_2012Metric_Pad1.20x1.40mm_HandSolder -> Resistor_SMD:R_0603_1608Metric_Pad0.98x0.95mm_HandSolder
- R2: value 100 -> R; footprint Resistor_SMD:R_0805_2012Metric_Pad1.20x1.40mm_HandSolder -> Resistor_SMD:R_0603_1608Metric_Pad0.98x0.95mm_HandSolder
- R20, R23, R26: value 500k -> 1k; footprint Resistor_SMD:R_0805_2012Metric_Pad1.20x1.40mm_HandSolder -> Resistor_SMD:R_0603_1608Metric_Pad0.98x0.95mm_HandSolder
- R29, R36: value 2k -> 4.7k
- R3: value 1k -> 8; footprint Resistor_SMD:R_0805_2012Metric_Pad1.20x1.40mm_HandSolder -> Resistor_SMD:R_0603_1608Metric_Pad0.98x0.95mm_HandSolder
- R30, R31: value R -> 10k; footprint Resistor_SMD:R_0805_2012Metric_Pad1.20x1.40mm_HandSolder -> Resistor_SMD:R_0603_1608Metric_Pad0.98x0.95mm_HandSolder
- R32: value R -> 10K; footprint Resistor_SMD:R_0805_2012Metric_Pad1.20x1.40mm_HandSolder -> Resistor_SMD:R_0603_1608Metric_Pad0.98x0.95mm_HandSolder
- R33: value 4.7k -> 10k
- R34: value 10K -> 2k
- R37, R38: value 10k -> 20R
- R4: value 8 -> R; footprint Resistor_SMD:R_0805_2012Metric_Pad1.20x1.40mm_HandSolder -> Resistor_SMD:R_0603_1608Metric_Pad0.98x0.95mm_HandSolder
- R6: value 1k -> R; footprint Resistor_SMD:R_0805_2012Metric_Pad1.20x1.40mm_HandSolder -> Resistor_SMD:R_0603_1608Metric_Pad0.98x0.95mm_HandSolder
- U2: value AMS1117-5.0 -> PC817; footprint Package_TO_SOT_SMD:SOT-223-3_TabPin2 -> Package_DIP:DIP-4_W7.62mm
- U3: value PC817 -> STM32F103C8Tx; footprint Package_DIP:DIP-4_W7.62mm -> Package_QFP:LQFP-48_7x7mm_P0.5mm
- U4: value TME-1205S -> XL1509-5.0; footprint Converter_DCDC:Converter_DCDC_TRACO_TME_03xxS_05xxS_12xxS_Single_THT -> Package_SO:SOIC-8_3.9x4.9mm_P1.27mm
- U5: value ESP32-C3_SUPERMINI_TH -> AMS1117-5.0; footprint ESP32-C3_SUPERMINI_TH:MODULE_ESP32-C3_SUPERMINI_TH -> Package_TO_SOT_SMD:SOT-223-3_TabPin2
- Y4: value 10M -> 32.768k; footprint Crystal:Crystal_SMD_5032-4Pin_5.0x3.2mm -> Crystal:Crystal_SMD_3215-2Pin_3.2x1.5mm
- moved LED_1 107.4 mm to (144.8, 181.5)
- moved R34 100.1 mm to (110.5, 154.0), turned to 0 degrees
- moved R35 95.5 mm to (110.5, 156.5), turned to 0 degrees
- moved D1 81.7 mm to (144.8, 172.3)
- moved J1 81.4 mm to (144.5, 111.1), turned to 180 degrees
- moved R29 79.8 mm to (106.2, 166.6)
- moved JP2 74.9 mm to (144.7, 153.2), turned to 0 degrees
- moved C4 70.6 mm to (146.0, 103.9)
- moved J5 69.0 mm to (104.7, 55.8)
- moved R31 68.5 mm to (88.0, 54.0)
- moved D2 67.1 mm to (144.6, 59.6)
- moved JP1 66.8 mm to (140.1, 153.2), turned to 0 degrees
- moved C21 63.3 mm to (91.5, 60.6), turned to 180 degrees
- moved J6 60.5 mm to (83.6, 57.9), turned to 90 degrees
- moved C20 58.5 mm to (91.3, 45.4), turned to 0 degrees
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Connections:
- C1 pad 1: /IAP -> /IBN
- C10 pad 1: /VCP -> /ICP
- C11 pad 1: Net-(U1-CLKIN) -> GND1
- C11 pad 2: GND1 -> /RESET
- C12 pad 1: Net-(U1-CLKOUT) -> Net-(JP1-A)
- C13 pad 1: Net-(JP5-A) -> Net-(JP1-A)
- C14 pad 1: Net-(JP5-A) -> GND1
- C14 pad 2: GND1 -> 3.3V
- C15 pad 1: Net-(U1-REFIN/OUT) -> GND1
- C15 pad 2: GND1 -> 3.3V
- C16 pad 1: Net-(U1-REFIN/OUT) -> Net-(JP3-A)
- C16 pad 2: GND1 -> 3.3V
- C19 pad 1: 3.3V -> Net-(U1-REFIN/OUT)
- C20 pad 1: 3.3V -> Net-(JP4-A)
- C20 pad 2: GND1 -> 3.3V
- C21 pad 1: +12V -> GND1
- C21 pad 2: GND -> 3.3V
- C22 pad 1: +12V -> Net-(U1-REFIN/OUT)
- C22 pad 2: GND -> GND1
- C23 pad 1: +5V -> Net-(U1-CLKIN)
- C24 pad 1: +5V -> Net-(U1-CLKOUT)
- C3 pad 1: /IBN -> /ICN
- C4 pad 1: /IBP -> /VN
- C5 pad 1: /ICN -> /VAP
- C6 pad 1: /ICP -> /VBP
- C7 pad 1: /VN -> /VCP
- C8 pad 1: /VAP -> /IAP
- C9 pad 1: /VBP -> /IBP
- D1 pad 1: GND1 -> /PA3
- D2 pad 1: /PA3 -> Net-(D2-K)
- D2 pad 2: Net-(D2-A) -> GNDPWR
- J1 pad 1: Net-(J1-Pin_1) -> /N
- J1 pad 2: Net-(J1-Pin_2) -> /C
- J4 pad 1: /N -> Net-(J4-Pin_1)
- J4 pad 2: /C -> Net-(J4-Pin_2)
- J5 pad 1: +12V -> /SWCLK
- J5 pad 2: GND -> /SWDIO
- J5 pad 3: (no net) -> GND1
- J6 pad 3: /I2C_SCL -> /I2C_SDA
- J6 pad 4: /I2C_SDA -> /I2C_SCL
- J9 pad A5: /SWDIO -> unconnected-(J9-CC1-PadA5)
- J9 pad A9: 3.3V -> +5V
- J9 pad B5: /SWCLK -> unconnected-(J9-CC2-PadB5)
- J9 pad B9: 3.3V -> +5V
- J9 pad SH: (no net) -> GND1
- JP1 pad 2: /BOOT -> +5V
- JP2 pad 1: Net-(JP2-A) -> Net-(JP1-A)
- JP2 pad 2: /BOOT2 -> 3.3V
- LED_ESP1 pad 1: Net-(LED_ESP1-K) -> /IO3
- R1 pad 1: GND1 -> Net-(J3-Pin_2)
- R1 pad 2: Net-(J1-Pin_1) -> GND1
- R10 pad 1: Net-(J2-Pin_1) -> GND1
- R10 pad 2: Net-(R10-Pad2) -> Net-(J4-Pin_1)
- R11 pad 1: Net-(R11-Pad1) -> /A
- R11 pad 2: /IBN -> /VAP
- R12 pad 1: Net-(R10-Pad2) -> /B
- R12 pad 2: /IBP -> /VBP
- R13 pad 1: Net-(J3-Pin_2) -> /C
- R13 pad 2: GND1 -> /VCP
- R14 pad 1: GND1 -> Net-(J2-Pin_2)
- R14 pad 2: Net-(J3-Pin_1) -> Net-(R14-Pad2)
- R15 pad 1: Net-(J3-Pin_2) -> Net-(J4-Pin_2)
- R16 pad 1: Net-(J3-Pin_1) -> Net-(J2-Pin_1)
- R17 pad 1: Net-(R15-Pad2) -> Net-(J3-Pin_1)
- R17 pad 2: /ICN -> Net-(R17-Pad2)
- R18 pad 1: Net-(R16-Pad2) -> Net-(J4-Pin_1)
- R18 pad 2: /ICP -> Net-(R18-Pad2)
- R19 pad 1: /N -> Net-(R19-Pad1)
- R19 pad 2: /VN -> /IBN
- R2 pad 1: Net-(J1-Pin_1) -> Net-(J2-Pin_2)
- R2 pad 2: Net-(R2-Pad2) -> Net-(J2-Pin_1)
- R20 pad 1: /A -> Net-(R14-Pad2)
- R20 pad 2: /VAP -> /IAN
- R22 pad 1: GND1 -> Net-(R16-Pad2)
- R22 pad 2: /VAP -> /IAP
- R23 pad 1: /B -> GND1
- R23 pad 2: /VBP -> /VAP
- R25 pad 2: /VBP -> /VCP
- R26 pad 1: /C -> Net-(R17-Pad2)
- R26 pad 2: /VCP -> /IBP
- R28 pad 1: GND1 -> Net-(R18-Pad2)
- R28 pad 2: /VCP -> /ICP
- R29 pad 1: Net-(D1-A) -> 3.3V
- R29 pad 2: 3.3V -> Net-(LED_1-A)
- R3 pad 1: Net-(R2-Pad2) -> Net-(J2-Pin_2)
- R3 pad 2: /IAP -> GND1
- R30 pad 1: Net-(J1-Pin_2) -> 3.3V
- R30 pad 2: Net-(J1-Pin_1) -> /RESET
- R31 pad 1: Net-(J2-Pin_2) -> Net-(JP3-A)
- R31 pad 2: Net-(J2-Pin_1) -> GND1
- R32 pad 1: Net-(J3-Pin_2) -> Net-(R32-Pad1)
- R32 pad 2: Net-(J3-Pin_1) -> Net-(U1-APCF)
- R33 pad 1: 3.3V -> Net-(JP4-A)
- R33 pad 2: Net-(LED_1-A) -> GND1
- R34 pad 1: Net-(R34-Pad1) -> 3.3V
- R34 pad 2: Net-(U1-APCF) -> /PA3
- R35 pad 1: Net-(D2-A) -> Net-(D1-A)
- R36 pad 1: 3.3V -> +5V
- R36 pad 2: /PA3 -> /PA12
- R37 pad 1: 3.3V -> /PA11
- R37 pad 2: /RESET -> Net-(J8-D--PadA7)
- R38 pad 1: Net-(JP2-A) -> /PA12
- R38 pad 2: GND1 -> Net-(J8-D+-PadA6)
- R39 pad 1: Net-(JP1-A) -> 3.3V
- R39 pad 2: GND1 -> /EN
- R4 pad 1: Net-(J1-Pin_2) -> Net-(J3-Pin_2)
- R4 pad 2: GND1 -> Net-(J3-Pin_1)
- R5 pad 1: Net-(J1-Pin_2) -> Net-(J4-Pin_2)
- R5 pad 2: Net-(R5-Pad2) -> GND1
- R6 pad 1: Net-(R5-Pad2) -> Net-(J4-Pin_2)
- R6 pad 2: /IAN -> Net-(J4-Pin_1)
- R7 pad 1: Net-(J2-Pin_2) -> GND1
- R7 pad 2: GND1 -> Net-(J2-Pin_1)
- R8 pad 2: Net-(J2-Pin_1) -> Net-(J3-Pin_1)
- R9 pad 1: Net-(J2-Pin_2) -> Net-(J3-Pin_2)
- R9 pad 2: Net-(R11-Pad1) -> Net-(R19-Pad1)
- U1 pad 3: Net-(JP5-A) -> Net-(JP1-A)
- U1 pad 4: Net-(JP5-A) -> Net-(JP1-A)
- U2 pad 1: GND1 -> Net-(R32-Pad1)
- U2 pad 2: 3.3V -> GND1
- U2 pad 3: +5V -> GND1
- U3 pad 1: Net-(R34-Pad1) -> 3.3V
- U3 pad 2: GND1 -> unconnected-(U3-PC13-Pad2)
- U3 pad 3: GND1 -> Net-(U3-PC14)
- U3 pad 4: /PA3 -> Net-(U3-PC15)
- U4 pad 1: GND -> +12V
- U4 pad 2: Net-(U4-+Vin) -> Net-(D2-K)
- U4 pad 3: Net-(U4--Vout) -> +5V
- U4 pad 4: +5V -> GNDPWR
- U5 pad 1: unconnected-(U5-GPIO1-Pad1) -> GND1
- U5 pad 2: unconnected-(U5-GPIO2-Pad2) -> 3.3V
- U5 pad 3: unconnected-(U5-GPIO3-Pad3) -> +5V
- Y2 pad 1: Net-(U10-PC15) -> Net-(U3-PC15)
- Y2 pad 2: Net-(U10-PC14) -> Net-(U3-PC14)
- Y3 pad 1: Net-(U10-PD1) -> Net-(U3-PD1)
- Y3 pad 3: Net-(U10-PD0) -> Net-(U3-PD0)
- Y4 pad 1: Net-(U1-CLKIN) -> Net-(C42-Pad2)
- Y4 pad 2: GND1 -> Net-(C39-Pad2)
Routing:
- net GND1: track 702.5 -> 96.3 mm, vias 2 -> 0
- net 3.3V: track 368.5 -> 7.10 mm, vias 3 -> 0
- net +5V: track 163.2 -> 6.82 mm
- net /ICP: track 58.6 -> 2.79 mm
- net /ICN: track 58.0 -> 2.85 mm
- net /SWDIO: track 53.9 -> 0.00 mm
- net /IBN: track 55.6 -> 2.73 mm
- net /IBP: track 55.6 -> 2.79 mm
- net /VCP: track 55.0 -> 3.00 mm
- net /VBP: track 54.1 -> 3.01 mm
- net /IAN: track 53.4 -> 2.85 mm
- net /VN: track 52.0 -> 1.51 mm
- net /IAP: track 53.0 -> 2.73 mm
- net /VAP: track 53.2 -> 3.00 mm
- net /SWCLK: track 47.5 -> 0.00 mm
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Other:
- board outline removed
- board text removed: "ESP32-S3"
- board text removed: "I2C"
- board text removed: "IAN"
- board text removed: "IAP"
- board text removed: "IBN"
- board text removed: "IBP"
- board text removed: "ICN"
- board text removed: "ICP"

Commit message: update 70%
Parts:
- removed JP1, JP2: Jumper_2_Open, Connector_PinHeader_2.54mm:PinHeader_1x02_P2.54mm_Vertical
- removed U2: PC817, Package_DIP:DIP-4_W7.62mm
- added Q1: Q_NPN_BEC, Package_TO_SOT_SMD:SOT-23, F.Cu at (85.9, 89.6)
- moved LED_1 130.0 mm to (98.2, 60.1)
- moved D4 113.1 mm to (117.5, 65.7), turned to 180 degrees
- moved TP3 109.2 mm to (130.2, 72.7)
- moved R29 108.8 mm to (98.1, 58.1)
- moved D1 105.2 mm to (86.1, 85.0)
- moved R46 93.6 mm to (116.3, 63.0), turned to 90 degrees
- moved TP1 88.4 mm to (150.6, 56.9)
- moved TP2 79.4 mm to (159.5, 56.9)
- moved R35 73.9 mm to (88.8, 85.9), turned to -90 degrees
- moved R34 71.5 mm to (85.9, 86.9), turned to 180 degrees
- moved C15 18.2 mm to (102.3, 71.7), turned to 90 degrees
- moved C17 16.4 mm to (100.8, 71.7), turned to 90 degrees
- moved C18 14.6 mm to (99.3, 71.7), turned to 90 degrees
- moved R16 5.10 mm to (93.2, 103.8)
- moved R22 5.10 mm to (93.2, 100.5)
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Connections:
- C12 pad 1: Net-(JP1-A) -> +5V
- C13 pad 1: Net-(JP1-A) -> +5V
- U1 pad 3: Net-(JP1-A) -> +5V
- U1 pad 4: Net-(JP1-A) -> +5V
- U3 pad 29: /UART1_RX -> unconnected-(U3-PA8-Pad29)
- U3 pad 30: /UART1_TX -> /UART1_RX
- U3 pad 31: /DIN -> /UART1_TX
Routing:
- net 3.3V: track 7.10 -> 109.0 mm
- net /VN: track 1.51 -> 45.9 mm
- net /VCP: track 3.00 -> 44.5 mm
- net /VBP: track 3.01 -> 40.6 mm
- net /VAP: track 3.00 -> 37.3 mm
- net GND1: track 96.3 -> 123.5 mm
- net /BOOT2: track 0.00 -> 25.2 mm, vias 0 -> 1
- net /EN: track 8.39 -> 33.1 mm, vias 0 -> 2
- net /PA12: track 0.00 -> 24.5 mm
- net /PA11: track 0.00 -> 24.1 mm
- net +5V: track 6.82 -> 24.1 mm
- net /ICN: track 2.85 -> 17.4 mm
- net /ICP: track 2.79 -> 15.6 mm
- net /BOOT: track 0.00 -> 12.4 mm, vias 0 -> 1
- net Net-(JP1-A): track 11.1 -> 0.00 mm
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
Commit message: upload 80%
Parts:
- J8, J9: footprint Connector_USB:USB_C_Receptacle_GCT_USB4110 -> Connector_USB:USB_C_Receptacle_Palconn_UTC16-G
- moved C29 59.3 mm to (149.6, 103.7)
- moved C33 58.3 mm to (163.1, 103.3), turned to 0 degrees
- moved J7 55.9 mm to (152.3, 106.4), turned to 90 degrees
- moved C30 50.1 mm to (144.2, 98.5)
- moved U4 46.0 mm to (154.2, 100.8), turned to 90 degrees
- moved L1 45.2 mm to (161.3, 96.5), turned to 0 degrees
- moved R42 41.4 mm to (163.1, 92.1), turned to 180 degrees
- moved D2 39.0 mm to (149.6, 98.3), turned to 90 degrees
- moved D3 38.6 mm to (147.9, 76.4), turned to 90 degrees
- moved LED1 32.4 mm to (154.9, 93.1), turned to 90 degrees
- moved TP1 32.1 mm to (143.7, 88.2)
- moved TP2 32.1 mm to (152.6, 88.2)
- moved U5 30.9 mm to (142.6, 76.3), turned to 90 degrees
- moved R40 28.8 mm to (127.9, 61.9)
- moved C31 28.8 mm to (152.1, 45.2)
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Connections:
- J1 pad 1: /N -> /A
- J1 pad 2: /C -> /B
- J1 pad 3: /B -> /C
- J1 pad 4: /A -> /N
Routing:
- net /VN: track 45.9 -> 10.9 mm
- net /VCP: track 44.5 -> 14.2 mm
- net /VBP: track 40.6 -> 15.7 mm
- net /VAP: track 37.3 -> 20.8 mm
- net /ICN: track 17.4 -> 2.79 mm
- net GND1: track 123.5 -> 137.1 mm
- net /ICP: track 15.6 -> 2.85 mm
- net /IAN: track 12.1 -> 2.73 mm
- net +5V: track 24.1 -> 31.5 mm
- net /IBP: track 9.94 -> 2.73 mm
- net /IAP: track 12.9 -> 6.18 mm
- net /IBN: track 9.39 -> 2.79 mm
- net +12V: track 21.7 -> 17.1 mm
- net GNDPWR: track 43.9 -> 47.5 mm
- net 3.3V: track 109.0 -> 111.9 mm
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Other:
- board outline added: 93 x 88 mm

Commit message: updat3 85%
Parts:
- moved TP3 33.8 mm to (154.2, 79.7)
- moved TP1 19.4 mm to (161.1, 79.7)
- moved TP2 16.7 mm to (167.0, 79.7)
- moved C13 6.03 mm to (99.2, 92.9)
- moved C20 6.03 mm to (96.5, 48.6)
- moved C21 6.03 mm to (96.7, 63.8)
- moved C22 6.03 mm to (116.9, 95.1)
- moved C23 6.03 mm to (109.9, 79.6)
- moved C24 6.03 mm to (104.1, 79.6)
- moved D1 6.03 mm to (91.2, 88.2)
- moved J5 6.03 mm to (107.7, 58.7)
- moved Q1 6.03 mm to (91.1, 92.8)
- moved R29 6.03 mm to (103.2, 61.3)
- moved R31 6.03 mm to (93.1, 57.2)
- moved R32 6.03 mm to (93.1, 95.9)
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Routing:
- net 3.3V: track 111.9 -> 240.4 mm, vias 0 -> 2
- net /UART1_TX: track 0.00 -> 37.2 mm
- net /UART1_RX: track 0.00 -> 36.8 mm
- net +5V: track 31.5 -> 61.0 mm
- net /VN: track 10.9 -> 38.3 mm
- net /VCP: track 14.2 -> 37.6 mm
- net /VBP: track 15.7 -> 35.6 mm
- net /IAN: track 2.73 -> 19.5 mm
- net GND1: track 137.1 -> 153.7 mm, vias 0 -> 36
- net /IAP: track 6.18 -> 20.2 mm
- net Net-(C40-Pad1): track 1.51 -> 15.4 mm, vias 0 -> 2
- net Net-(C43-Pad1): track 1.51 -> 14.4 mm
- net /VAP: track 20.8 -> 33.3 mm
- net /I2C_SCL: track 7.01 -> 15.9 mm, vias 0 -> 1
- net /IBP: track 2.73 -> 10.8 mm
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- added copper zone on F.Cu, net 3.3V
- added copper zone on B.Cu, net GND1
- added copper zone on F.Cu, net GND1
- added copper zone on B.Cu, net GNDPWR
- added copper zone on F.Cu, net GNDPWR
